File: hardware/boysenboard.kicad_sch (KiCad schematic)
At the start: 97 parts, among them J1 1050171001, J2 54-00164, J3 NPTC101KFXC-RC, J4 NPTC081KFXC-RC, J5 Micro-SD, J6 NPTC081KFXC-RC, J7 NPTC061KFXC-RC, Q1 BSS308PEH6327XTSA1, SW1 PTS645SL70SMTR92LFS, U1 F1C200s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

Commit message: Fixed footprint references and kicad 5->6 models
Parts:
- C3, C7: footprint licheeduino:CP_EIA-3216-18_Kemet-A -> boysenboard:CP_EIA-3216-18_Kemet-A
- D1: footprint licheeduino:D_SOD-123F -> boysenboard:D_SOD-123F
- D2, D3, D4, D5, D6: footprint licheeduino:LED_1206_3216Metric_Castellated -> boysenboard:LED_1206_3216Metric_Castellated
- F1: footprint licheeduino:Fuse_1206_3216Metric_Castellated -> boysenboard:Fuse_1206_3216Metric_Castellated
- H1, H2, H3, H4: footprint licheeduino:mounting_hole_125mil -> boysenboard:mounting_hole_125mil
- J1: footprint licheeduino:USB_Micro-B_Molex-105017-0001 -> boysenboard:USB_Micro-B_Molex-105017-0001
- J2: footprint licheeduino:barrel_jack_2.1mm -> boysenboard:barrel_jack_2.1mm
- J5: footprint licheedunio:micro-sd -> boysenboard:micro-sd
- SW1: footprint licheeduino:switch_tactile_6x6mm_smt -> boysenboard:switch_tactile_6x6mm_smt
- TP1, TP2, TP3, TP4, TP5: footprint licheeduino:test_point_RCSCTE -> boysenboard:test_point_RCSCTE
- U1: footprint licheedunio:QFN-88 -> boysenboard:QFN-88
